File: UTCPW_MountingBoard.kicad_pcb (KiCad board)
At the start: 2 copper layers, 38.1 x 35.6 mm, 8 parts, among them U1 UTCPW_SampleStrip

Commit message: Updated the /net of pads so they connect to /GND
Was worried at first that the solder paste layer is blocking the drill hole views in the render plot. But for fabrication it shouldn't matter.
Updated the drill holes of the adapter so that they are connected to the big chunk of metal on both sides of the board.
Connections:
- REF** pad : (no net) -> /GND (x3)
Routing:
- added copper zone on B.Cu, net /GND
- removed copper zone on B.Cu, net (none)
Changed lines of the file:
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@@
     (fp_circle (center 1.2192 -1.7526) (end 1.6256 -1.7526) (layer "Dwgs.User") (width 0.0508) (fill none))
     (fp_circle (center -1.2192 -1.7526) (end -0.8128 -1.7526) (layer "Dwgs.User") (width 0.0508) (fill none))
-    (pad "" thru_hole circle (at -1.2192 -3.9624) (size 1.2192 1.2192) (drill 1.143) (layers *.Cu *.Mask))
-    (pad "" thru_hole circle (at 1.2192 -3.9624) (size 1.2192 1.2192) (drill 1.143) (layers *.Cu *.Mask))
-    (pad "" thru_hole circle (at 1.2192 -1.7526) (size 1.2192 1.2192) (drill 1.143) (layers *.Cu *.Mask))
-    (pad "" thru_hole circle (at -1.2192 -1.7526) (size 1.2192 1.2192) (drill 1.143) (layers *.Cu *.Mask))
+    (pad "" thru_hole circle (at -1.2192 -3.9624) (size 1.2192 1.2192) (drill 1.143) (layers *.Cu *.Mask)
+      (net 5 "/GND"))
+    (pad "" thru_hole circle (at 1.2192 -3.9624) (size 1.2192 1.2192) (drill 1.143) (layers *.Cu *.Mask)
+      (net 5 "/GND"))
+    (pad "" thru_hole circle (at 1.2192 -1.7526) (size 1.2192 1.2192) (drill 1.143) (layers *.Cu *.Mask)
+      (net 5 "/GND"))
+    (pad "" thru_hole circle (at -1.2192 -1.7526) (size 1.2192 1.2192) (drill 1.143) (layers *.Cu *.Mask)
+      (net 5 "/GND"))
     (pad "1" smd rect (at 0 -2.7686) (size 0.4064 5.5372) (layers "F.Cu" "F.Mask")
       (net 2 "/Dev3"))
@@
     (fp_circle (center 1.2192 -1.7526) (end 1.6256 -1.7526) (layer "Dwgs.User") (width 0.0508) (fill none))
     (fp_circle (center -1.2192 -3.9624) (end -0.8128 -3.9624) (layer "Dwgs.User") (width 0.0508) (fill none))
-    (pad "" thru_hole circle (at -1.2192 -1.7526) (size 1.2192 1.2192) (drill 1.143) (layers *.Cu *.Mask))
-    (pad "" thru_hole circle (at 1.2192 -1.7526) (size 1.2192 1.2192) (drill 1.143) (layers *.Cu *.Mask))
-    (pad "" thru_hole circle (at -1.2192 -3.9624) (size 1.2192 1.2192) (drill 1.143) (layers *.Cu *.Mask))
-    (pad "" thru_hole circle (at 1.2192 -3.9624) (size 1.2192 1.2192) (drill 1.143) (layers *.Cu *.Mask))
+    (pad "" thru_hole circle (at -1.2192 -1.7526) (size 1.2192 1.2192) (drill 1.143) (layers *.Cu *.Mask)
+      (net 5 "/GND"))
+    (pad "" thru_hole circle (at 1.2192 -1.7526) (size 1.2192 1.2192) (drill 1.143) (layers *.Cu *.Mask)
+      (net 5 "/GND"))
+    (pad "" thru_hole circle (at -1.2192 -3.9624) (size 1.2192 1.2192) (drill 1.143) (layers *.Cu *.Mask)
+      (net 5 "/GND"))
+    (pad "" thru_hole circle (at 1.2192 -3.9624) (size 1.2192 1.2192) (drill 1.143) (layers *.Cu *.Mask)
+      (net 5 "/GND"))
     (pad "1" smd rect (at 0 -2.7686) (size 0.4064 5.5372) (layers "F.Cu" "F.Mask")
       (net 4 "/Dev1"))
@@
     (fp_circle (center 1.2192 -1.7526) (end 1.6256 -1.7526) (layer "Dwgs.User") (width 0.0508) (fill none))
     (fp_circle (center 1.2192 -3.9624) (end 1.6256 -3.9624) (layer "Dwgs.User") (width 0.0508) (fill none))
-    (pad "" thru_hole circle (at -1.2192 -1.7526) (size 1.2192 1.2192) (drill 1.143) (layers *.Cu *.Mask))
-    (pad "" thru_hole circle (at -1.2192 -3.9624) (size 1.2192 1.2192) (drill 1.143) (layers *.Cu *.Mask))
-    (pad "" thru_hole circle (at 1.2192 -1.7526) (size 1.2192 1.2192) (drill 1.143) (layers *.Cu *.Mask))
-    (pad "" thru_hole circle (at 1.2192 -3.9624) (size 1.2192 1.2192) (drill 1.143) (layers *.Cu *.Mask))
+    (pad "" thru_hole circle (at -1.2192 -1.7526) (size 1.2192 1.2192) (drill 1.143) (layers *.Cu *.Mask)
+      (net 5 "/GND"))
+    (pad "" thru_hole circle (at -1.2192 -3.9624) (size 1.2192 1.2192) (drill 1.143) (layers *.Cu *.Mask)
+      (net 5 "/GND"))
+    (pad "" thru_hole circle (at 1.2192 -1.7526) (size 1.2192 1.2192) (drill 1.143) (layers *.Cu *.Mask)
+      (net 5 "/GND"))
+    (pad "" thru_hole circle (at 1.2192 -3.9624) (size 1.2192 1.2192) (drill 1.143) (layers *.Cu *.Mask)
+      (net 5 "/GND"))
     (pad "1" smd rect (at 0 -2.7686) (size 0.4064 5.5372) (layers "F.Cu" "F.Mask")
       (net 1 "/Dev2"))
@@
   (segment (start 114.3 114.3) (end 117.348 111.252) (width 0.3302) (layer "F.Cu") (net 4))
   (zone (net 5) (net_name "/GND") (layer "F.Cu") (hatch edge 0.508)
-    (connect_pads yes (clearance 0.254))
-    (min_thickness 0.254) (filled_areas_thickness no)
+    (connect_pads yes (clearance 0.1524))
+    (min_thickness 0.1524) (filled_areas_thickness no)
     (fill yes (thermal_gap 0.508) (thermal_bridge_width 0.508))
     (polygon
@@
     )
   )
-  (zone (net 0) (net_name "") (layer "B.Cu") (hatch edge 0.508)
+  (zone (net 5) (net_name "/GND") (layer "B.Cu") (hatch edge 0.508)
     (connect_pads yes (clearance 0.127))
     (min_thickness 0.254) (filled_areas_thickness no)
